Commit message: deneme öncesi

File: urdf/robot.urdf copy.xacro (robot description, xacro)
@@ -102,5 +102,5 @@
     <origin xyz="0 0 -0.0099" rpy="0 0 0"/>
     <axis xyz="-0.6534 -0.5970 0.0"/>
-    <limit lower="0" upper="1.57" effort="10.0" velocity="1.0"/>
+    <limit lower="0" upper="2.0" effort="10.0" velocity="1.0"/>
     <dynamics damping="2.0" friction="0.5"/>
   </joint>
@@ -142,6 +142,6 @@
     <child link="link3"/>
     <origin xyz="-0.1322 0.1533 -0.0337" rpy="0 0 0"/>
-    <axis xyz="-0.6534 -0.5570 0"/>
-    <limit lower="0" upper="1.57" effort="10.0" velocity="1.0"/>
+    <axis xyz="0 0 1"/>
+    <limit lower="0" upper="2.0" effort="10.0" velocity="1.0"/>
     <dynamics damping="2.0" friction="0.5"/>
   </joint>
@@ -154,9 +154,9 @@
     </visual>
     <collision>
-      <origin xyz="0.05 -0.03 0" rpy="0 0 0"/>
+      <origin xyz="0.1947 -0.0906 0.2727" rpy="0 0 0"/>
       <geometry><box size="0.06 0.04 0.04"/></geometry>
     </collision>
     <inertial>
-      <origin xyz="0.05 -0.03 0" rpy="0 0 0"/>
+      <origin xyz="0.1947 -0.0906 0.2727" rpy="0 0 0"/>
       <mass value="0.15"/>
       <inertia ixx="0.0002" ixy="0" ixz="0" iyy="0.0002" iyz="0" izz="0.0001"/>
@@ -172,19 +172,19 @@
   <link name="gripper_link">
     <visual>
-      <origin xyz="0.1947 -0.0906 0.2627" rpy="0 0 0"/>
+      <origin xyz="0.1947 -0.0906 0.2727" rpy="0 0 0"/>
       <geometry><mesh filename="package://3dof_rrr_robot_arm/meshes/gripper.stl" scale="0.001 0.001 0.001"/></geometry>
       <material name="Brown"/>
     </visual>
     <visual>
-      <origin xyz="0.1947 -0.0906 0.2627" rpy="0 0 0"/>
+      <origin xyz="0.1947 -0.0906 0.2727" rpy="0 0 0"/>
       <geometry><mesh filename="package://3dof_rrr_robot_arm/meshes/kapak_new.stl" scale="0.001 0.001 0.001"/></geometry>
       <material name="Grey"/>
     </visual>
     <collision>
-      <origin xyz="0 0 0.08" rpy="0 0 0"/>
+      <origin xyz="0.1947 -0.0906 0.35" rpy="0 0 0"/>
       <geometry><box size="0.04 0.06 0.1"/></geometry>
     </collision>
     <inertial>
-      <origin xyz="0 0 0.08" rpy="0 0 0"/>
+      <origin xyz="0.1947 -0.0906 0.35" rpy="0 0 0"/>
       <mass value="0.1"/>
       <inertia ixx="0.0001" ixy="0" ixz="0" iyy="0.0001" iyz="0" izz="0.00005"/>
