Commit message: Refactor: modular controller configs with xacro
- Added separate yaml configs for position/velocity/effort controllers
- Converted URDF to xacro with parameterized transmissions
- Hardware interface now set from yaml via launch argument
- Removed MoveIt dependencies
- Single launch file supports all controller types

File: urdf/robot.urdf.xacro (robot description, xacro)
@@ -1,4 +1,21 @@
 <?xml version="1.0"?>
-<robot name="3DoF_RRR_Robot_Arm">
+<robot name="3DoF_RRR_Robot_Arm" xmlns:xacro="http://www.ros.org/wiki/xacro">
+  <!-- Hardware Interface Argument (from yaml or launch) -->
+  <xacro:arg name="hw_interface" default="PositionJointInterface"/>
+  <xacro:property name="hw_interface" value="$(arg hw_interface)"/>
+  <!-- Transmission Macro -->
+  <xacro:macro name="joint_transmission" params="joint_name">
+    <transmission name="trans_${joint_name}">
+      <type>transmission_interface/SimpleTransmission</type>
+      <joint name="${joint_name}">
+        <hardwareInterface>hardware_interface/${hw_interface}</hardwareInterface>
+      </joint>
+      <actuator name="motor_${joint_name}">
+        <hardwareInterface>hardware_interface/${hw_interface}</hardwareInterface>
+        <mechanicalReduction>1</mechanicalReduction>
+      </actuator>
+    </transmission>
+  </xacro:macro>
+  <!-- Materials -->
   <material name="Red"><color rgba="1.0 0.0 0.0 1.0"/></material>
   <material name="Green"><color rgba="0.0 1.0 0.0 1.0"/></material>
@@ -12,4 +29,5 @@
   <material name="Brown"><color rgba="0.6 0.3 0.0 1.0"/></material>
   <material name="Grey"><color rgba="0.5 0.5 0.5 1.0"/></material>
+  <!-- World link -->
   <link name="world"/>
   <joint name="world_to_base" type="fixed">
@@ -18,4 +36,5 @@
     <origin xyz="0 0 0" rpy="3.14159 0 0"/>
   </joint>
+  <!-- Base Link -->
   <link name="base_link">
     <visual>
@@ -25,8 +44,14 @@
     </visual>
     <collision>
-      <origin xyz="0 0 0" rpy="0 0 0"/>
-      <geometry><mesh filename="package://3dof_rrr_robot_arm/meshes/base_part2.stl" scale="0.001 0.001 0.001"/></geometry>
-    </collision>
-  </link>
+      <origin xyz="0 0 -0.03" rpy="0 0 0"/>
+      <geometry><box size="0.08 0.08 0.06"/></geometry>
+    </collision>
+    <inertial>
+      <origin xyz="0 0 -0.03" rpy="0 0 0"/>
+      <mass value="0.5"/>
+      <inertia ixx="0.001" ixy="0" ixz="0" iyy="0.001" iyz="0" izz="0.001"/>
+    </inertial>
+  </link>
+  <!-- Joint 1 -->
   <joint name="joint1" type="revolute">
     <parent link="base_link"/>
@@ -35,5 +60,7 @@
     <axis xyz="0 0 1"/>
     <limit lower="-2.268" upper="2.268" effort="10.0" velocity="1.0"/>
-  </joint>
+    <dynamics damping="0.5" friction="0.1"/>
+  </joint>
+  <!-- Link 1 -->
   <link name="link1">
     <visual>
@@ -57,5 +84,15 @@
       <material name="Cyan"/>
     </visual>
-  </link>
+    <collision>
+      <origin xyz="0 0 0.05" rpy="0 0 0"/>
+      <geometry><cylinder radius="0.04" length="0.12"/></geometry>
+    </collision>
+    <inertial>
+      <origin xyz="0 0 0.05" rpy="0 0 0"/>
+      <mass value="0.3"/>
+      <inertia ixx="0.0005" ixy="0" ixz="0" iyy="0.0005" iyz="0" izz="0.0003"/>
+    </inertial>
+  </link>
+  <!-- Joint 2 -->
   <joint name="joint2" type="revolute">
     <parent link="link1"/>
@@ -64,5 +101,7 @@
     <axis xyz="-0.6534 -0.5970 0.0"/>
     <limit lower="0" upper="1.57" effort="10.0" velocity="1.0"/>
-  </joint>
+    <dynamics damping="0.5" friction="0.1"/>
+  </joint>
+  <!-- Link 2 -->
   <link name="link2">
     <visual>
@@ -86,5 +125,15 @@
       <material name="Pink"/>
     </visual>
-  </link>
+    <collision>
+      <origin xyz="-0.05 0.05 0" rpy="0 1.57 0"/>
+      <geometry><cylinder radius="0.025" length="0.15"/></geometry>
+    </collision>
+    <inertial>
+      <origin xyz="-0.05 0.05 0" rpy="0 0 0"/>
+      <mass value="0.2"/>
+      <inertia ixx="0.0003" ixy="0" ixz="0" iyy="0.0003" iyz="0" izz="0.0002"/>
+    </inertial>
+  </link>
+  <!-- Joint 3 -->
   <joint name="joint3" type="revolute">
     <parent link="link2"/>
@@ -93,5 +142,7 @@
     <axis xyz="-0.6534 -0.5570 0"/>
     <limit lower="0" upper="1.57" effort="10.0" velocity="1.0"/>
-  </joint>
+    <dynamics damping="0.5" friction="0.1"/>
+  </joint>
+  <!-- Link 3 -->
   <link name="link3">
     <visual>
@@ -100,5 +151,15 @@
       <material name="Lime"/>
     </visual>
-  </link>
+    <collision>
+      <origin xyz="0.05 -0.03 0" rpy="0 0 0"/>
+      <geometry><box size="0.06 0.04 0.04"/></geometry>
+    </collision>
+    <inertial>
+      <origin xyz="0.05 -0.03 0" rpy="0 0 0"/>
+      <mass value="0.15"/>
+      <inertia ixx="0.0002" ixy="0" ixz="0" iyy="0.0002" iyz="0" izz="0.0001"/>
+    </inertial>
+  </link>
+  <!-- Gripper Joint -->
   <joint name="gripper_joint" type="fixed">
     <parent link="link3"/>
@@ -106,4 +167,5 @@
     <origin xyz="0 0 0" rpy="0 0 0"/>
   </joint>
+  <!-- Gripper Link -->
   <link name="gripper_link">
     <visual>
@@ -117,5 +179,15 @@
       <material name="Grey"/>
     </visual>
-  </link>
+    <collision>
+      <origin xyz="0 0 0.08" rpy="0 0 0"/>
+      <geometry><box size="0.04 0.06 0.1"/></geometry>
+    </collision>
+    <inertial>
+      <origin xyz="0 0 0.08" rpy="0 0 0"/>
+      <mass value="0.1"/>
+      <inertia ixx="0.0001" ixy="0" ixz="0" iyy="0.0001" iyz="0" izz="0.00005"/>
+    </inertial>
+  </link>
+  <!-- Tool Tip Joint -->
   <joint name="tool_tip_joint" type="fixed">
     <parent link="gripper_link"/>
@@ -123,4 +195,5 @@
     <origin xyz="-0.05 0.06 0.2" rpy="0 0 0"/>
   </joint>
+  <!-- Tool Tip Link -->
   <link name="tool_tip">
     <visual>
@@ -128,4 +201,43 @@
       <material name="Green"/>
     </visual>
-  </link>
+    <collision>
+      <geometry><sphere radius="0.012"/></geometry>
+    </collision>
+    <inertial>
+      <mass value="0.01"/>
+      <inertia ixx="0.000001" ixy="0" ixz="0" iyy="0.000001" iyz="0" izz="0.000001"/>
+    </inertial>
+  </link>
+  <!-- ==================== GAZEBO SPECIFIC ==================== -->
+  <!-- Gazebo Colors -->
+  <gazebo reference="base_link">
+    <material>Gazebo/Red</material>
+  </gazebo>
+  <gazebo reference="link1">
+    <material>Gazebo/Blue</material>
+  </gazebo>
+  <gazebo reference="link2">
+    <material>Gazebo/Purple</material>
+  </gazebo>
+  <gazebo reference="link3">
+    <material>Gazebo/Green</material>
+  </gazebo>
+  <gazebo reference="gripper_link">
+    <material>Gazebo/Orange</material>
+  </gazebo>
+  <gazebo reference="tool_tip">
+    <material>Gazebo/Green</material>
+  </gazebo>
+  <!-- ros_control plugin -->
+  <gazebo>
+    <plugin name="gazebo_ros_control" filename="libgazebo_ros_control.so">
+      <robotNamespace>/</robotNamespace>
+      <robotSimType>gazebo_ros_control/DefaultRobotHWSim</robotSimType>
+      <legacyModeNS>true</legacyModeNS>
+    </plugin>
+  </gazebo>
+  <!-- Transmissions (uses hw_interface from argument) -->
+  <xacro:joint_transmission joint_name="joint1"/>
+  <xacro:joint_transmission joint_name="joint2"/>
+  <xacro:joint_transmission joint_name="joint3"/>
 </robot>

Commit message: optimize edilmeye hazir

File: urdf/robot.urdf.xacro (robot description, xacro)
@@ -18,15 +18,17 @@
   </xacro:macro>
   <!-- Materials -->
-  <material name="Red"><color rgba="1.0 0.0 0.0 1.0"/></material>
-  <material name="Green"><color rgba="0.0 1.0 0.0 1.0"/></material>
-  <material name="Blue"><color rgba="0.0 0.0 1.0 1.0"/></material>
-  <material name="Yellow"><color rgba="1.0 1.0 0.0 1.0"/></material>
-  <material name="Cyan"><color rgba="0.0 1.0 1.0 1.0"/></material>
-  <material name="Magenta"><color rgba="1.0 0.0 1.0 1.0"/></material>
-  <material name="Orange"><color rgba="1.0 0.5 0.0 1.0"/></material>
-  <material name="Lime"><color rgba="0.5 1.0 0.0 1.0"/></material>
-  <material name="Pink"><color rgba="1.0 0.07 0.57 1.0"/></material>
-  <material name="Brown"><color rgba="0.6 0.3 0.0 1.0"/></material>
-  <material name="Grey"><color rgba="0.5 0.5 0.5 1.0"/></material>
+  <material name="Black"><color rgba="0.1 0.1 0.1 1.0"/></material>
+  <material name="DarkGrey"><color rgba="0.2 0.2 0.2 1.0"/></material>
+  <material name="Red"><color rgba="0.1 0.1 0.1 1.0"/></material>
+  <material name="Green"><color rgba="0.1 0.1 0.1 1.0"/></material>
+  <material name="Blue"><color rgba="0.15 0.15 0.15 1.0"/></material>
+  <material name="Yellow"><color rgba="0.2 0.2 0.2 1.0"/></material>
+  <material name="Cyan"><color rgba="0.15 0.15 0.15 1.0"/></material>
+  <material name="Magenta"><color rgba="0.1 0.1 0.1 1.0"/></material>
+  <material name="Orange"><color rgba="0.2 0.2 0.2 1.0"/></material>
+  <material name="Lime"><color rgba="0.15 0.15 0.15 1.0"/></material>
+  <material name="Pink"><color rgba="0.1 0.1 0.1 1.0"/></material>
+  <material name="Brown"><color rgba="0.1 0.1 0.1 1.0"/></material>
+  <material name="Grey"><color rgba="0.2 0.2 0.2 1.0"/></material>
   <!-- World link -->
   <link name="world"/>
@@ -60,5 +62,5 @@
     <axis xyz="0 0 1"/>
     <limit lower="-2.268" upper="2.268" effort="10.0" velocity="1.0"/>
-    <dynamics damping="0.5" friction="0.1"/>
+    <dynamics damping="2.0" friction="0.5"/>
   </joint>
   <!-- Link 1 -->
@@ -101,5 +103,5 @@
     <axis xyz="-0.6534 -0.5970 0.0"/>
     <limit lower="0" upper="1.57" effort="10.0" velocity="1.0"/>
-    <dynamics damping="0.5" friction="0.1"/>
+    <dynamics damping="2.0" friction="0.5"/>
   </joint>
   <!-- Link 2 -->
@@ -142,10 +144,10 @@
     <axis xyz="-0.6534 -0.5570 0"/>
     <limit lower="0" upper="1.57" effort="10.0" velocity="1.0"/>
-    <dynamics damping="0.5" friction="0.1"/>
+    <dynamics damping="2.0" friction="0.5"/>
   </joint>
   <!-- Link 3 -->
   <link name="link3">
     <visual>
-      <origin xyz="0.1947 -0.0906 0.2627" rpy="0 0 0"/>
+      <origin xyz="0.1947 -0.0906 0.2727" rpy="0 0 0"/>
       <geometry><mesh filename="package://3dof_rrr_robot_arm/meshes/servo_2.stl" scale="0.001 0.001 0.001"/></geometry>
       <material name="Lime"/>
@@ -210,22 +212,22 @@
   </link>
   <!-- ==================== GAZEBO SPECIFIC ==================== -->
-  <!-- Gazebo Colors -->
+  <!-- Gazebo Colors - All Black/Dark -->
   <gazebo reference="base_link">
+    <material>Gazebo/Black</material>
+  </gazebo>
+  <gazebo reference="link1">
+    <material>Gazebo/DarkGrey</material>
+  </gazebo>
+  <gazebo reference="link2">
+    <material>Gazebo/Black</material>
+  </gazebo>
+  <gazebo reference="link3">
+    <material>Gazebo/DarkGrey</material>
+  </gazebo>
+  <gazebo reference="gripper_link">
+    <material>Gazebo/Black</material>
+  </gazebo>
+  <gazebo reference="tool_tip">
     <material>Gazebo/Red</material>
-  </gazebo>
-  <gazebo reference="link1">
-    <material>Gazebo/Blue</material>
-  </gazebo>
-  <gazebo reference="link2">
-    <material>Gazebo/Purple</material>
-  </gazebo>
-  <gazebo reference="link3">
-    <material>Gazebo/Green</material>
-  </gazebo>
-  <gazebo reference="gripper_link">
-    <material>Gazebo/Orange</material>
-  </gazebo>
-  <gazebo reference="tool_tip">
-    <material>Gazebo/Green</material>
   </gazebo>
   <!-- ros_control plugin -->

Commit message: teste_hazir

File: urdf/robot.urdf.xacro (robot description, xacro)
@@ -197,15 +197,9 @@
     <origin xyz="-0.05 0.06 0.2" rpy="0 0 0"/>
   </joint>
-  <!-- Tool Tip Link -->
+  <!-- Tool Tip Link (invisible - just for reference frame) -->
   <link name="tool_tip">
-    <visual>
-      <geometry><sphere radius="0.012"/></geometry>
-      <material name="Green"/>
-    </visual>
-    <collision>
-      <geometry><sphere radius="0.012"/></geometry>
-    </collision>
-    <inertial>
-      <mass value="0.01"/>
+    <!-- Visual removed - soldering effect will be spawned here -->
+    <inertial>
+      <mass value="0.001"/>
       <inertia ixx="0.000001" ixy="0" ixz="0" iyy="0.000001" iyz="0" izz="0.000001"/>
     </inertial>

Commit message: calismayan_guncel_versiyon

File: urdf/robot.urdf.xacro (robot description, xacro)
@@ -102,5 +102,5 @@
     <origin xyz="0 0 -0.0099" rpy="0 0 0"/>
     <axis xyz="-0.6534 -0.5970 0.0"/>
-    <limit lower="0" upper="1.57" effort="10.0" velocity="1.0"/>
+    <limit lower="0" upper="2.0" effort="10.0" velocity="1.0"/>
     <dynamics damping="2.0" friction="0.5"/>
   </joint>
@@ -143,5 +143,5 @@
     <origin xyz="-0.1322 0.1533 -0.0337" rpy="0 0 0"/>
     <axis xyz="-0.6534 -0.5570 0"/>
-    <limit lower="0" upper="1.57" effort="10.0" velocity="1.0"/>
+    <limit lower="0" upper="2.0" effort="10.0" velocity="1.0"/>
     <dynamics damping="2.0" friction="0.5"/>
   </joint>
@@ -154,9 +154,9 @@
     </visual>
     <collision>
-      <origin xyz="0.05 -0.03 0" rpy="0 0 0"/>
+      <origin xyz="0.1947 -0.0906 0.2727" rpy="0 0 0"/>
       <geometry><box size="0.06 0.04 0.04"/></geometry>
     </collision>
     <inertial>
-      <origin xyz="0.05 -0.03 0" rpy="0 0 0"/>
+      <origin xyz="0.1947 -0.0906 0.2727" rpy="0 0 0"/>
       <mass value="0.15"/>
       <inertia ixx="0.0002" ixy="0" ixz="0" iyy="0.0002" iyz="0" izz="0.0001"/>
@@ -172,19 +172,19 @@
   <link name="gripper_link">
     <visual>
-      <origin xyz="0.1947 -0.0906 0.2627" rpy="0 0 0"/>
+      <origin xyz="0.1947 -0.0906 0.2727" rpy="0 0 0"/>
       <geometry><mesh filename="package://3dof_rrr_robot_arm/meshes/gripper.stl" scale="0.001 0.001 0.001"/></geometry>
       <material name="Brown"/>
     </visual>
     <visual>
-      <origin xyz="0.1947 -0.0906 0.2627" rpy="0 0 0"/>
+      <origin xyz="0.1947 -0.0906 0.2727" rpy="0 0 0"/>
       <geometry><mesh filename="package://3dof_rrr_robot_arm/meshes/kapak_new.stl" scale="0.001 0.001 0.001"/></geometry>
       <material name="Grey"/>
     </visual>
     <collision>
-      <origin xyz="0 0 0.08" rpy="0 0 0"/>
+      <origin xyz="0.1947 -0.0906 0.35" rpy="0 0 0"/>
       <geometry><box size="0.04 0.06 0.1"/></geometry>
     </collision>
     <inertial>
-      <origin xyz="0 0 0.08" rpy="0 0 0"/>
+      <origin xyz="0.1947 -0.0906 0.35" rpy="0 0 0"/>
       <mass value="0.1"/>
       <inertia ixx="0.0001" ixy="0" ixz="0" iyy="0.0001" iyz="0" izz="0.00005"/>

Commit message: vallahi_cok_fena_oldu_her_sey_Hazir

File: urdf/robot.urdf.xacro (robot description, xacro)
@@ -102,6 +102,6 @@
     <origin xyz="0 0 -0.0099" rpy="0 0 0"/>
     <axis xyz="-0.6534 -0.5970 0.0"/>
-    <limit lower="0" upper="1.57" effort="10.0" velocity="1.0"/>
-    <dynamics damping="2.0" friction="0.5"/>
+    <limit lower="0" upper="2.0" effort="10.0" velocity="1.0"/>
+    <dynamics damping="0.8" friction="0.2"/>
   </joint>
   <!-- Link 2 -->
@@ -129,5 +129,5 @@
     <collision>
       <origin xyz="-0.05 0.05 0" rpy="0 1.57 0"/>
-      <geometry><cylinder radius="0.025" length="0.15"/></geometry>
+      <geometry><cylinder radius="0.015" length="0.15"/></geometry>
     </collision>
     <inertial>
@@ -143,5 +143,5 @@
     <origin xyz="-0.1322 0.1533 -0.0337" rpy="0 0 0"/>
     <axis xyz="-0.6534 -0.5570 0"/>
-    <limit lower="0" upper="1.57" effort="10.0" velocity="1.0"/>
+    <limit lower="0" upper="2.0" effort="10.0" velocity="1.0"/>
     <dynamics damping="2.0" friction="0.5"/>
   </joint>
@@ -215,10 +215,13 @@
   <gazebo reference="link2">
     <material>Gazebo/Black</material>
+    <self_collide>false</self_collide>
   </gazebo>
   <gazebo reference="link3">
     <material>Gazebo/DarkGrey</material>
+    <self_collide>false</self_collide>
   </gazebo>
   <gazebo reference="gripper_link">
     <material>Gazebo/Black</material>
+    <self_collide>false</self_collide>
   </gazebo>
   <gazebo reference="tool_tip">
